Commit message: Subida inicial con mis modificaciones

File: description/lidar.xacro (robot description, xacro)
@@ -9,10 +9,10 @@
         <parent link="chasis"/>
         <child link="lidar_frame"/>
-        <origin xyz="${lidar_offset_x} 0.0 ${lidar_offset_z}" rpy="0 0 ${pi}"/>
+        <origin xyz="0.1 0 0.175" rpy="0 0 ${pi}"/>
     </joint>
     <link name="lidar_frame">
         <visual>
             <geometry>
-                <cylinder radius="${lidar_radius}" length="${lidar_thickness}"/>
+                <cylinder radius="0.05" length="0.04"/>
             </geometry>
             <material name="orange"/>
@@ -20,8 +20,8 @@
         <collision>
             <geometry>
-                <cylinder radius="${lidar_radius}" length="${lidar_thickness}"/>
+                <cylinder radius="0.05" length="0.04"/>
             </geometry>
         </collision>
-        <xacro:inertial_cylinder mass="0.1" radius="${lidar_radius}" length="${lidar_thickness}">
+        <xacro:inertial_cylinder mass="0.1" radius="0.05" length="0.04">
             <origin xyz="0 0 0" rpy="0 0 0"/>
         </xacro:inertial_cylinder>

File: description/robot_main.xacro (robot description, xacro)
@@ -2,14 +2,14 @@
 <robot xmlns:xacro="http://www.ros.org/wiki/xacro">
     <xacro:include filename = "inertial_macros.xacro" />
-    <xacro:property name="chassis_length"           value="0.320"/>
-    <xacro:property name="chassis_width"            value="0.240"/>
-    <xacro:property name="chassis_height"           value="0.078"/>
-    <xacro:property name="chassis_mass"             value="0.700"/>
+    <xacro:property name="chassis_length"           value="0.360"/>
+    <xacro:property name="chassis_width"            value="0.250"/>
+    <xacro:property name="chassis_height"           value="0.150"/>
+    <xacro:property name="chassis_mass"             value="0.500"/>
     <xacro:property name="wheel_radius"             value="0.034"/>
-    <xacro:property name="wheel_thickness"          value="0.026"/>
-    <xacro:property name="wheel_mass"               value="0.050"/>
-    <xacro:property name="wheel_offset_x"           value="0.133"/>
-    <xacro:property name="wheel_offset_y"           value="0.133"/>
-    <xacro:property name="wheel_offset_z"           value="0.020"/>
+    <xacro:property name="wheel_thickness"          value="0.030"/>
+    <xacro:property name="wheel_mass"               value="0.100"/>
+    <xacro:property name="wheel_offset_x"           value="0"/>
+    <xacro:property name="wheel_offset_y"           value="0.135"/>
+    <xacro:property name="wheel_offset_z"           value="0"/>
     <xacro:property name="caster_wheel_radius"      value="${wheel_radius - wheel_offset_z}"/>
     <xacro:property name="caster_wheel_mass"        value="0.010"/>
@@ -48,22 +48,22 @@
         <parent link= "base_link"/>
         <child link= "chasis"/>
-        <origin xyz= "${-wheel_offset_x} 0 ${-wheel_offset_z}"/>
+        <origin xyz= "-0.1 0 0"/>
     </joint>
     <link name="chasis">
         <visual>
-            <origin xyz= "${chassis_length/2} 0 ${chassis_height/2}" rpy= "0 0 0"/>
+            <origin xyz= "0.18 0 0.075" rpy= "0 0 0"/>
             <geometry>
-                <box size = "${chassis_length} ${chassis_width} ${chassis_height}"/>
+                <box size = "0.36 0.25 0.15"/>
             </geometry>
             <material name= "black"/>
         </visual>
         <collision>
-            <origin xyz= "${chassis_length/2} 0 ${chassis_height/2}" rpy= "0 0 0"/>
+            <origin xyz= "0.18 0 0.075" rpy= "0 0 0"/>
             <geometry>
-                <box size = "${chassis_length} ${chassis_width} ${chassis_height}"/>
+                <box size = "0.36 0.26 0.15"/>
             </geometry>
         </collision>
-        <xacro:inertial_box mass= "0.5" x="${chassis_length}" y="${chassis_width}" z="${chassis_height}">
-            <origin xyz= "${chassis_length/2} 0 ${chassis_height/2}" rpy= "0 0 0"/>
+        <xacro:inertial_box mass= "0.5" x="0.36" y="0.26" z="0.15">
+            <origin xyz= "0.18 0 0.075" rpy= "0 0 0"/>
         </xacro:inertial_box>
     </link>
@@ -75,5 +75,5 @@
         <parent link= "base_link"/>
         <child link= "left_wheel"/>
-        <origin xyz= "0 ${wheel_offset_y} 0" rpy = "${pi/2} 0 0"/>
+        <origin xyz= "0 0.135 0" rpy = "${pi/2} 0 0"/>
         <axis xyz= "0 0 -1"/>
     </joint>
@@ -81,5 +81,5 @@
         <visual>
             <geometry>
-                <cylinder radius = "${wheel_radius}" length= "${wheel_thickness}"/>
+                <cylinder radius = "0.034" length= "0.03"/>
             </geometry>
             <material name= "orange"/>
@@ -87,8 +87,8 @@
         <collision>
             <geometry>
-                <sphere radius = "${wheel_radius}" />
+                <sphere radius = "0.034" />
             </geometry>
         </collision>
-        <xacro:inertial_cylinder mass = "${wheel_mass}" radius= "${wheel_radius}" length= "${wheel_thickness}">
+        <xacro:inertial_cylinder mass = "0.1" radius= "0.034" length= "0.03">
             <origin xyz= "0 0 0" rpy= "0 0 0"/>
         </xacro:inertial_cylinder>
@@ -101,5 +101,5 @@
         <parent link= "base_link"/>
         <child link= "right_wheel"/>
-        <origin xyz= "0 ${-wheel_offset_y} 0" rpy = "${pi/2} 0 0"/>
+        <origin xyz= "0 -0.135 0" rpy = "${pi/2} 0 0"/>
         <axis xyz= "0 0 -1"/>
     </joint>
@@ -107,5 +107,5 @@
         <visual>
             <geometry>
-                <cylinder radius = "${wheel_radius}" length= "${wheel_thickness}"/>
+                <cylinder radius = "0.034" length= "0.03"/>
             </geometry>
             <material name= "orange"/>
@@ -113,8 +113,8 @@
         <collision>
             <geometry>
-                <sphere radius = "${wheel_radius}" />
+                <sphere radius = "0.034" />
             </geometry>
         </collision>
-        <xacro:inertial_cylinder mass = "${wheel_mass}" radius= "${wheel_radius}" length= "${wheel_thickness}">
+        <xacro:inertial_cylinder mass = "0.1" radius= "0.034" length= "0.03">
             <origin xyz= "0 0 0" rpy= "0 0 0"/>
         </xacro:inertial_cylinder>
@@ -127,10 +127,10 @@
         <parent link= "chasis"/>
         <child link= "caster_wheel"/>
-        <origin xyz= "${caster_wheel_offset_x} 0 0"/>
+        <origin xyz= "0.30 0 0"/>
     </joint>
     <link name="caster_wheel">
         <visual>
             <geometry>
-                <sphere radius = "${caster_wheel_radius}"/>
+                <sphere radius = "0.025"/>
             </geometry>
             <material name= "orange"/>
@@ -138,8 +138,8 @@
         <collision>
             <geometry>
-                <sphere radius = "${caster_wheel_radius}"/>
+                <sphere radius = "0.025"/>
             </geometry>
         </collision>
-        <xacro:inertial_sphere mass= "${caster_wheel_mass}" radius= "${caster_wheel_radius}">
+        <xacro:inertial_sphere mass= "0.1" radius= "0.025">
             <origin xyz= "0 0 0" rpy= "0 0 0"/>
         </xacro:inertial_sphere>

File: description/ros2_control.xacro (robot description, xacro)
@@ -9,7 +9,7 @@
                     <param name="loop_rate">30</param>
                     <param name="device">/dev/ttyUSB1</param>
-                    <param name="baud_rate">115200</param>
+                    <param name="baud_rate">57600</param>
                     <param name="timeout_ms">1000</param>
-                    <param name="enc_counts_per_rev">616</param>
+                    <param name="enc_counts_per_rev">1976</param>
             </hardware>
             <joint name="left_wheel_joint">

Commit message: jun 8 modificaciones

File: description/lidar.xacro (robot description, xacro)
@@ -1,18 +1,18 @@
 <?xml version="1.0"?>
 <robot xmlns:xacro="http://www.ros.org/wiki/xacro" name="robot">
-    <xacro:property name="lidar_radius"             value="0.025"/>
-    <xacro:property name="lidar_thickness"          value="0.040"/>
-    <xacro:property name="lidar_offset_x"           value="0.230"/>
-    <xacro:property name="lidar_offset_z"           value="0.098"/>
+    <xacro:property name="lidar_radius"             value="0.035"/>
+    <xacro:property name="lidar_thickness"          value="0.050"/>
+    <xacro:property name="lidar_offset_x"           value="0.185"/>
+    <xacro:property name="lidar_offset_z"           value="0.180"/>
     <!-- Lidar -->
     <joint name="lidar_joint" type="fixed">
         <parent link="chasis"/>
         <child link="lidar_frame"/>
-        <origin xyz="0.1 0 0.175" rpy="0 0 ${pi}"/>
+        <origin xyz="${lidar_offset_x} 0.0 ${lidar_offset_z}" rpy="0 0 ${pi}"/>
     </joint>
     <link name="lidar_frame">
         <visual>
             <geometry>
-                <cylinder radius="0.05" length="0.04"/>
+                <cylinder radius="${lidar_radius}" length="${lidar_thickness}"/>
             </geometry>
             <material name="orange"/>
@@ -20,8 +20,8 @@
         <collision>
             <geometry>
-                <cylinder radius="0.05" length="0.04"/>
+                <cylinder radius="${lidar_radius}" length="${lidar_thickness}"/>
             </geometry>
         </collision>
-        <xacro:inertial_cylinder mass="0.1" radius="0.05" length="0.04">
+        <xacro:inertial_cylinder mass="0.1" radius="${lidar_radius}" length="${lidar_thickness}">
             <origin xyz="0 0 0" rpy="0 0 0"/>
         </xacro:inertial_cylinder>

File: description/robot_main.xacro (robot description, xacro)
@@ -3,16 +3,16 @@
     <xacro:include filename = "inertial_macros.xacro" />
     <xacro:property name="chassis_length"           value="0.360"/>
-    <xacro:property name="chassis_width"            value="0.250"/>
-    <xacro:property name="chassis_height"           value="0.150"/>
-    <xacro:property name="chassis_mass"             value="0.500"/>
-    <xacro:property name="wheel_radius"             value="0.034"/>
-    <xacro:property name="wheel_thickness"          value="0.030"/>
-    <xacro:property name="wheel_mass"               value="0.100"/>
-    <xacro:property name="wheel_offset_x"           value="0"/>
-    <xacro:property name="wheel_offset_y"           value="0.135"/>
-    <xacro:property name="wheel_offset_z"           value="0"/>
-    <xacro:property name="caster_wheel_radius"      value="${wheel_radius - wheel_offset_z}"/>
+    <xacro:property name="chassis_width"            value="0.270"/>
+    <xacro:property name="chassis_height"           value="0.170"/>
+    <xacro:property name="chassis_mass"             value="0.700"/>
+    <xacro:property name="wheel_radius"             value="0.033"/>
+    <xacro:property name="wheel_thickness"          value="0.026"/>
+    <xacro:property name="wheel_mass"               value="0.050"/>
+    <xacro:property name="wheel_offset_x"           value="0.100"/>
+    <xacro:property name="wheel_offset_y"           value="0.148"/>
+    <xacro:property name="wheel_offset_z"           value="0.01"/>
+    <xacro:property name="caster_wheel_radius"      value="0.015"/>
     <xacro:property name="caster_wheel_mass"        value="0.010"/>
-    <xacro:property name="caster_wheel_offset_x"    value="0.230"/>
+    <xacro:property name="caster_wheel_offset_x"    value="0.299"/>
     <xacro:property name="caster_wheel_offset_z"    value="${wheel_offset_z - wheel_radius + caster_wheel_radius}"/>
     <!-- Colors -->
@@ -48,22 +48,22 @@
         <parent link= "base_link"/>
         <child link= "chasis"/>
-        <origin xyz= "-0.1 0 0"/>
+        <origin xyz= "${-wheel_offset_x} 0 ${-wheel_offset_z}"/>
     </joint>
     <link name="chasis">
         <visual>
-            <origin xyz= "0.18 0 0.075" rpy= "0 0 0"/>
+            <origin xyz= "${chassis_length/2} 0 ${chassis_height/2}" rpy= "0 0 0"/>
             <geometry>
-                <box size = "0.36 0.25 0.15"/>
+                <box size = "${chassis_length} ${chassis_width} ${chassis_height}"/>
             </geometry>
             <material name= "black"/>
         </visual>
         <collision>
-            <origin xyz= "0.18 0 0.075" rpy= "0 0 0"/>
+            <origin xyz= "${chassis_length/2} 0 ${chassis_height/2}" rpy= "0 0 0"/>
             <geometry>
-                <box size = "0.36 0.26 0.15"/>
+                <box size = "${chassis_length} ${chassis_width} ${chassis_height}"/>
             </geometry>
         </collision>
-        <xacro:inertial_box mass= "0.5" x="0.36" y="0.26" z="0.15">
-            <origin xyz= "0.18 0 0.075" rpy= "0 0 0"/>
+        <xacro:inertial_box mass= "0.5" x="${chassis_length}" y="${chassis_width}" z="${chassis_height}">
+            <origin xyz= "${chassis_length/2} 0 ${chassis_height/2}" rpy= "0 0 0"/>
         </xacro:inertial_box>
     </link>
@@ -75,5 +75,5 @@
         <parent link= "base_link"/>
         <child link= "left_wheel"/>
-        <origin xyz= "0 0.135 0" rpy = "${pi/2} 0 0"/>
+        <origin xyz= "0 ${wheel_offset_y} 0" rpy = "${pi/2} 0 0"/>
         <axis xyz= "0 0 -1"/>
     </joint>
@@ -81,5 +81,5 @@
         <visual>
             <geometry>
-                <cylinder radius = "0.034" length= "0.03"/>
+                <cylinder radius = "${wheel_radius}" length= "${wheel_thickness}"/>
             </geometry>
             <material name= "orange"/>
@@ -87,8 +87,8 @@
         <collision>
             <geometry>
-                <sphere radius = "0.034" />
+                <sphere radius = "${wheel_radius}" />
             </geometry>
         </collision>
-        <xacro:inertial_cylinder mass = "0.1" radius= "0.034" length= "0.03">
+        <xacro:inertial_cylinder mass = "${wheel_mass}" radius= "${wheel_radius}" length= "${wheel_thickness}">
             <origin xyz= "0 0 0" rpy= "0 0 0"/>
         </xacro:inertial_cylinder>
@@ -101,5 +101,5 @@
         <parent link= "base_link"/>
         <child link= "right_wheel"/>
-        <origin xyz= "0 -0.135 0" rpy = "${pi/2} 0 0"/>
+        <origin xyz= "0 ${-wheel_offset_y} 0" rpy = "${pi/2} 0 0"/>
         <axis xyz= "0 0 -1"/>
     </joint>
@@ -107,5 +107,5 @@
         <visual>
             <geometry>
-                <cylinder radius = "0.034" length= "0.03"/>
+                <cylinder radius = "${wheel_radius}" length= "${wheel_thickness}"/>
             </geometry>
             <material name= "orange"/>
@@ -113,8 +113,8 @@
         <collision>
             <geometry>
-                <sphere radius = "0.034" />
+                <sphere radius = "${wheel_radius}" />
             </geometry>
         </collision>
-        <xacro:inertial_cylinder mass = "0.1" radius= "0.034" length= "0.03">
+        <xacro:inertial_cylinder mass = "${wheel_mass}" radius= "${wheel_radius}" length= "${wheel_thickness}">
             <origin xyz= "0 0 0" rpy= "0 0 0"/>
         </xacro:inertial_cylinder>
@@ -127,10 +127,10 @@
         <parent link= "chasis"/>
         <child link= "caster_wheel"/>
-        <origin xyz= "0.30 0 0"/>
+        <origin xyz= "${caster_wheel_offset_x} 0 0"/>
     </joint>
     <link name="caster_wheel">
         <visual>
             <geometry>
-                <sphere radius = "0.025"/>
+                <sphere radius = "${caster_wheel_radius}"/>
             </geometry>
             <material name= "orange"/>
@@ -138,8 +138,8 @@
         <collision>
             <geometry>
-                <sphere radius = "0.025"/>
+                <sphere radius = "${caster_wheel_radius}"/>
             </geometry>
         </collision>
-        <xacro:inertial_sphere mass= "0.1" radius= "0.025">
+        <xacro:inertial_sphere mass= "${caster_wheel_mass}" radius= "${caster_wheel_radius}">
             <origin xyz= "0 0 0" rpy= "0 0 0"/>
         </xacro:inertial_sphere>
